File: hardware/waft_frontpanel.kicad_pcb (KiCad board)
At the start: 2 copper layers, 30.5 x 128.5 mm, 12 parts

Commit message: Rev 1.0 Sent for fabrication
Parts:
- removed the G*** at (72.5, 28.8)
- added G***: LOGO, europi:WaftFrontPanelSolderMask, F.Cu at (67.8, 88.8)
- added G***: LOGO, europi:WaftFrontPanelTopCopper, F.Cu at (67.8, 88.8)
- moved ? 0.09 mm to (60.0, 135.7)
- moved ? 0.09 mm to (75.4, 135.7)
Routing:
- net (no net): track 0.00 -> 104.5 mm
Other:
- outline, holes or cut-outs redrawn
- net class Default: trace_width 0.25 -> 0.4
- net class double added: clearance 0.2, trace_width 0.5, via_dia 0.6, via_drill 0.4
